File: tnc.sch (KiCad schematic (older format))
At the start: 55 parts, among them CON1 PJ2030D, K1 MK12C02, P1 CONN_3X2, P2 CONN_2, Q1 BC847C, SW1 SW_PUSH, U1 HC-05, U2 APE8800N, U3 BU33TD3WG, U4 ATMEGA328P-A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

Commit message: Update component vaues
Signed-off-by: Angel Hitov <angelhitov@gmail.com>
Parts:
- C1, C16, C17, C22, C23, C3, C4, C8, C9: value C -> 100nF
- C10, C11, C13, C14, C18, C20, C21: value C -> 100pF
- C15, C24: value CP1 -> 10uF
- C5: value C -> 10nF
- C6, C7: value C -> 10pF
- D1: value LED -> Blue LED
- FB1, FB2, FB3, FB4: value FILTER -> BLM21PG331SN1D
- P1: value CONN_3X2 -> ISP
- R1, R11, R12, R15, R8: value R -> 10k
- R10, R16: value R -> 1k
- R13, R9: value R -> n/a
- R14, R2: value R -> 0
- R3: value R -> 8k2
- R4: value R -> 100k
- R5: value R -> 15k
- R6, R7: value R -> 1M
- U4: value ATMEGA328P-A -> ATMEGA328P-AU
- X1: value CRYSTAL_SMD -> QKT-3225SMD 16.0000MHz
