File: bttnc2.kicad_pcb (KiCad board)
At the start: 2 copper layers, 70 x 40 mm, 105 parts, among them K1 MK12C02, P1 ISP, P2 BATTERY, P3 SMA, P4 USB_OTG, P5 U.FL, P6 Serial, Q1 MMBT3904, SW1 SW_PUSH, U1 HC-05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

Commit message: Update schematics and pcb
Parts:
- moved D8 0.53 mm to (115.9, 118.1)
Routing:
- net GND: track 292.7 -> 300.8 mm, vias 76 -> 77
- net (no net): vias 1 -> 0
Other:
- board text added: "APRS Bluetooth TNC tracker rev. 0.2a"
- board text added: "Battery"
- board text added: "GND"
- board text added: "LZ1ARM"
- board text added: "RX"
- board text added: "TX"
