File: bttnc2.kicad_pcb (KiCad board)
At the start: 2 copper layers, 70 x 40 mm, 105 parts, among them K1 MK12C02, P1 ISP, P2 BATTERY, P3 SMA, P4 USB_OTG, P5 U.FL, P6 Serial, Q1 MMBT3904, SW1 SW_PUSH, U1 HC-05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

Commit message: Update component values in PCB and export BOM
Parts:
- C10, C19, C2, C20, C25, C26, C29, C31: value C -> 100nF
- C11: value CP1 -> 100uF
- C12, C18: value C -> 20pF
- C13, C14: value C -> 36pF
- C21: value CP1 -> 100nF
- C27, C30, C32: value CP1 -> 10uF
- C33, C34: value C -> DNI
- D10, D11, D5, D6, D7, D9: value D_Schottky -> BAT42
- D2: value LED -> Green LED
- D4: value LED -> Red LED
- L1, L3: value INDUCTOR -> 56nH
- L2: value INDUCTOR -> 68nH
- R11, R20, R21, R8: value R -> 100k
- R12: value R -> 100
- R13: value R -> 1.2k
- R14, R17, R18, R23: value R -> 1k
- R19, R22, R25: value R -> 10k
- R28: value R -> 0

Commit message: Update elements values
This values was changed at device bring up.
We have working hardware configuration.
Parts:
- C28: value C -> 100nF
- D2: value Green LED -> Red LED
- D3: value LED -> Green LED
- D4: value Red LED -> Green LED
- D6: value BAT42 -> DNI
- D8: value LED -> Blue LED
- FB2: value BLM21PG331SN1D -> DNI
- R2: value 0 -> DNI
- R24: value R -> 1k
- R26: value R -> 0
- R27: value R -> DNI
- R9: value n/a -> DNI
Changed lines of the file:
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@@
       (effects (font (size 0.5 0.5) (thickness 0.125)))
     )
-    (fp_text value "Green LED" (at 7.3406 -0.0508 180) (layer F.Fab)
+    (fp_text value "Red LED" (at 7.3406 -0.0508 180) (layer F.Fab)
       (effects (font (size 0.5 0.5) (thickness 0.125)))
     )
@@
       (effects (font (size 1 1) (thickness 0.15)))
     )
-    (fp_text value LED (at -1.7526 1.651 270) (layer F.Fab)
+    (fp_text value "Green LED" (at -1.7526 1.651 270) (layer F.Fab)
       (effects (font (size 1 1) (thickness 0.15)))
     )
@@
       (effects (font (size 0.5 0.5) (thickness 0.125)))
     )
-    (fp_text value "Red LED" (at 5.8166 1.651 360) (layer F.Fab)
+    (fp_text value "Green LED" (at 5.8166 1.651 360) (layer F.Fab)
       (effects (font (size 0.5 0.5) (thickness 0.125)))
     )
@@
       (effects (font (size 1 1) (thickness 0.15)) (justify mirror))
     )
-    (fp_text value BLM21PG331SN1D (at 1.397 -7.62 180) (layer B.Fab)
+    (fp_text value DNI (at 1.397 -7.62 180) (layer B.Fab)
       (effects (font (size 1 1) (thickness 0.15)) (justify mirror))
     )
@@
       (effects (font (size 1 1) (thickness 0.15)))
     )
-    (fp_text value 0 (at -2.032 -1.651 360) (layer F.Fab)
+    (fp_text value DNI (at -2.032 -1.651 360) (layer F.Fab)
       (effects (font (size 1 1) (thickness 0.15)))
     )
@@
       (effects (font (size 1 1) (thickness 0.15)) (justify mirror))
     )
-    (fp_text value n/a (at 6.9088 -0.3048) (layer B.Fab)
+    (fp_text value DNI (at 6.9088 -0.3048) (layer B.Fab)
       (effects (font (size 1 1) (thickness 0.15)) (justify mirror))
     )
@@
       (effects (font (size 1 1) (thickness 0.15)) (justify mirror))
     )
-    (fp_text value BAT42 (at -1.524 5.6515 90) (layer B.Fab)
+    (fp_text value DNI (at -1.524 5.6515 90) (layer B.Fab)
       (effects (font (size 1 1) (thickness 0.15)) (justify mirror))
     )
@@
       (effects (font (size 1 1) (thickness 0.15)) (justify mirror))
     )
-    (fp_text value C (at 6.0452 -0.1016 270) (layer B.Fab)
+    (fp_text value 100nF (at 6.0452 -0.1016 270) (layer B.Fab)
       (effects (font (size 1 1) (thickness 0.15)) (justify mirror))
     )
@@
       (effects (font (size 1 1) (thickness 0.15)))
     )
-    (fp_text value LED (at -2.8448 -0.6096 180) (layer F.Fab)
+    (fp_text value "Blue LED" (at -2.8448 -0.6096 180) (layer F.Fab)
       (effects (font (size 1 1) (thickness 0.15)))
     )
@@
       (effects (font (size 1 1) (thickness 0.15)) (justify mirror))
     )
-    (fp_text value R (at -1.016 -5.08 180) (layer B.Fab)
+    (fp_text value 1k (at -1.016 -5.08 180) (layer B.Fab)
       (effects (font (size 1 1) (thickness 0.15)) (justify mirror))
     )
@@
       (effects (font (size 1 1) (thickness 0.15)))
     )
-    (fp_text value R (at -0.889 -1.6002) (layer F.Fab)
+    (fp_text value 0 (at -0.889 -1.6002) (layer F.Fab)
       (effects (font (size 1 1) (thickness 0.15)))
     )
@@
       (effects (font (size 1 1) (thickness 0.15)) (justify mirror))
     )
-    (fp_text value R (at -1.0668 3.3528 270) (layer B.Fab)
-      (effects (font (size 1 1) (thickness 0.15)) (justify mirror))
-    )
+    (fp_text value DNI (at -1.0668 3.3528 270) (layer B.Fab)
+      (effects (font (size 1 1) (thickness 0.15)) (justify mirror))
+    )
