File: bttnc2.sch (KiCad schematic (older format))
At the start: 72 parts, among them K1 MK12C02, P1 ISP, P2 BATTERY, P3 BNC, P4 USB_OTG, SW1 SW_PUSH, U1 HC-05, U2 APE8800N, U3 BU33TD3WG, U4 ATMEGA328P-AU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

Commit message: Update bttnc project. Sch and Pcb files.
Parts:
- removed R11, R8: R, Resistors_SMD:R_0805, symbol R-RESCUE-bttnc2
- added C25, C26, C28, C29, C31: C, Capacitors_SMD:C_0805, symbol C
- added C27, C30, C32: CP1, Capacitors_SMD:C_1206, symbol CP1
- added D10, D11, D5, D6, D7, D9: D_Schottky, Diodes_SMD:MiniMELF_Standard, symbol D_Schottky
- added D8: LED, LEDs:LED_0805, symbol LED
- added Q1: MMBT3904, TO_SOT_Packages_SMD:SOT-23, symbol MMBT3904
- added R11, R19, R20, R21, R22, R23, R24, R25, R26, R27, R8: R, Resistors_SMD:R_0805, symbol R
- added U10: Quectel-L80, footprints:Qectel-L80, symbol Quectel-L80
- added U11: FDG6342L, TO_SOT_Packages_SMD:SC-70-6, symbol FDG6342L
- added U9: LM358, SMD_Packages:SOIC-8-N, symbol LM358
- P3: footprint SMD_Packages:SOIC-8-N -> footprints:CON-SMA-EDGE
- SW1: footprint footprints:B3FS-1002P -> Buttons_Switches_ThroughHole:SW_Tactile_SPST_Angled
Connections:
- net labels added: GPS_EN, GPS_RESET, RXD, TXD
- net labels removed: RF_RXD, RF_TXD
- wire segments 194 -> 237

Commit message: Sch update - missing changes
Connections:
- wire segments 237 -> 285

Commit message: Latest updates
Parts:
- C21: footprint Capacitors_SMD:C_1210 -> Capacitors_SMD:C_0805
- D8: symbol LED -> LED-RESCUE-bttnc2
- P4: symbol USB_OTG -> USB_OTG-RESCUE-bttnc2
Connections:
- wire segments 285 -> 240
Other:
- moved on the sheet: C19
Changed lines of the file:
@@
 U 1 1 5620161C
 P 8150 4500
-F 0 "K1" H 8200 4200 60  0000 C CNN
+F 0 "K1" V 8250 4350 60  0000 C CNN
 F 1 "MK12C02" H 8000 4650 60  0000 C CNN
 F 2 "footprints:MK12C02" H 8150 4500 60  0001 C CNN
@@
 F 0 "C21" H 9100 2800 50  0000 L CNN
 F 1 "CP1" H 9100 2600 50  0000 L CNN
-F 2 "Capacitors_SMD:C_1210" H 9050 2700 60  0001 C CNN
+F 2 "Capacitors_SMD:C_0805" H 9050 2700 60  0001 C CNN
 F 3 "~" H 9050 2700 60  0000 C CNN
 	1    9050 2700
@@
 $EndComp
 $Comp
-L GND-RESCUE-bttnc2 #PWR032
-U 1 1 582A2D87
-P 9300 4200
-F 0 "#PWR032" H 9300 4200 30  0001 C CNN
-F 1 "GND" H 9300 4130 30  0001 C CNN
-F 2 "" H 9300 4200 60  0000 C CNN
-F 3 "" H 9300 4200 60  0000 C CNN
-	1    9300 4200
-	0    -1   -1   0
-$EndComp
-$Comp
 L R-RESCUE-bttnc2 R13
 U 1 1 582A5589
@@
 L C-RESCUE-bttnc2 C19
 U 1 1 582A784C
-P 8250 4900
-F 0 "C19" H 8250 5000 40  0000 L CNN
-F 1 "C" H 8256 4815 40  0000 L CNN
-F 2 "Capacitors_SMD:C_0805" H 8288 4750 30  0001 C CNN
-F 3 "~" H 8250 4900 60  0000 C CNN
-	1    8250 4900
+P 8650 4950
+F 0 "C19" H 8650 5050 40  0000 L CNN
+F 1 "C" H 8656 4865 40  0000 L CNN
+F 2 "Capacitors_SMD:C_0805" H 8688 4800 30  0001 C CNN
+F 3 "~" H 8650 4950 60  0000 C CNN
+	1    8650 4950
 	1    0    0    -1
 $EndComp
@@
 $EndComp
 $Comp
-L USB_OTG P4
+L USB_OTG-RESCUE-bttnc2 P4
 U 1 1 5831006C
 P 10050 2650
@@
 F 0 "Q1" H 12800 1175 50  0000 L CNN
 F 1 "MMBT3904" H 12800 1100 50  0000 L CNN
-F 2 "TO_SOT_Packages_SMD:SOT-23" H 12800 1025 50  0000 L CIN
+F 2 "TO_SOT_Packages_SMD:SOT-23" H 12800 1025 50  0001 L CIN
 F 3 "" H 12600 1100 50  0000 L CNN
 	1    12600 1100
@@
 GPS_RESET
 $Comp
-L LED D8
+L LED-RESCUE-bttnc2 D8
 U 1 1 5847BE44
 P 12900 1250
@@
 	1    0    0    -1
 $EndComp
+$Comp
+L GND #PWR052
+U 1 1 5855596B
+P 8650 5150
+F 0 "#PWR052" H 8650 4900 50  0001 C CNN
+F 1 "GND" H 8650 5000 50  0000 C CNN
+F 2 "" H 8650 5150 50  0000 C CNN
+F 3 "" H 8650 5150 50  0000 C CNN
+	1    8650 5150
+	1    0    0    -1
+$EndComp
 Wire Wire Line
 	3150 4500 3600 4500
@@
 	6450 3550 6450 3950
 Wire Wire Line
-	1250 4700 1250 4800
-Wire Wire Line
-	1250 4800 1250 4900
+	1250 4700 1250 4900
 Wire Wire Line
 	1100 5300 1100 4800
@@
 Connection ~ 1250 4800
 Wire Wire Line
-	1250 2000 1250 2500
-Wire Wire Line
-	1250 2500 1250 2600
-Wire Wire Line
-	1250 2600 1250 2700
-Wire Wire Line
-	1250 2700 1250 2900
+	1250 2000 1250 2900
 Connection ~ 1250 2600
 Connection ~ 1250 2900
@@
 	3650 3300 3650 3550
 Wire Wire Line
-	1900 1950 1900 2000
-Wire Wire Line
-	1900 2000 1900 2150
-Wire Wire Line
-	1900 2150 1900 2250
+	1900 1950 1900 2250
 Wire Wire Line
 	1900 2000 1800 2000
@@
 	750  2500 700  2500
 Wire Wire Line
-	700  2500 700  2700
-Wire Wire Line
-	700  2700 700  2900
+	700  2500 700  2900
 Wire Wire Line
 	700  2900 750  2900
@@
 	4800 7550 4800 7500
 Wire Wire Line
-	4300 7500 4300 7550
-Wire Wire Line
-	4300 7550 4300 7650
+	4300 7500 4300 7650
 Connection ~ 4300 7550
 Wire Wire Line
 	3800 7050 3800 7100
 Wire Wire Line
-	4750 7050 4800 7050
-Wire Wire Line
-	4800 7050 5150 7050
+	4750 7050 5150 7050
 Wire Wire Line
 	4800 7050 4800 7100
@@
 	800  750  700  750
 Wire Wire Line
-	1300 750  1350 750
-Wire Wire Line
-	1350 750  1400 750
+	1300 750  1400 750
 Wire Wire Line
 	1900 750  2000 750
@@
 	3900 3550 3650 3550
 Wire Wire Line
-	4000 3250 4300 3250
-Wire Wire Line
-	4300 3250 4400 3250
+	4000 3250 4400 3250
 Wire Wire Line
 	1300 2000 1250 2000
 Connection ~ 1250 2000
 Wire Wire Line
-	2450 2150 2600 2150
-Wire Wire Line
-	2600 2150 2700 2150
+	2450 2150 2700 2150
 Connection ~ 2600 2150
 Wire Wire Line
@@
 	1650 7050 1550 7050
 Wire Wire Line
-	1550 6700 1550 7050
-Wire Wire Line
-	1550 7050 1550 7100
+	1550 6700 1550 7100
 Wire Wire Line
 	1550 7500 1550 7550
 Wire Wire Line
-	1550 7550 2100 7550
-Wire Wire Line
-	2100 7550 2650 7550
+	1550 7550 2650 7550
 Wire Wire Line
 	2650 7550 2650 7500
 Wire Wire Line
-	2100 7500 2100 7550
-Wire Wire Line
-	2100 7550 2100 7650
+	2100 7500 2100 7650
 Connection ~ 2100 7550
 Wire Wire Line
-	1150 7200 1300 7200
-Wire Wire Line
-	1300 7200 1650 7200
+	1150 7200 1650 7200
 Wire Wire Line
 	1300 6700 1550 6700
@@
 Connection ~ 3900 3550
 Wire Wire Line
-	4300 2950 4300 3250
-Wire Wire Line
-	4300 3250 4300 3550
+	4300 2950 4300 3550
 Connection ~ 4300 3250
 Wire Wire Line
@@
 	7000 1250 7250 1250
 Wire Wire Line
-	8150 1750 8150 1850
-Wire Wire Line
-	8150 1850 8150 2000
+	8150 1750 8150 2000
 Connection ~ 8150 1850
 Wire Wire Line
 	7000 1350 7250 1350
 Wire Wire Line
-	8150 1150 8200 1150
-Wire Wire Line
-	8200 1150 8500 1150
-Wire Wire Line
-	8500 1150 8600 1150
+	8150 1150 8600 1150
 Connection ~ 8200 1150
 Connection ~ 8500 1150
@@
 	10300 1550 10300 2000
 Wire Wire Line
-	8500 2450 8500 3150
-Wire Wire Line
-	8500 3150 8500 3400
-Wire Wire Line
-	8500 3400 8500 3650
+	8500 2450 8500 3650
 Wire Wire Line
 	8800 3550 9400 3550
@@
 Connection ~ 8500 3650
 Wire Wire Line
-	8500 4650 8500 4700
-Wire Wire Line
-	3500 7550 3800 7550
-Wire Wire Line
-	3800 7550 4300 7550
-Wire Wire Line
-	4300 7550 4800 7550
-Wire Wire Line
-	4800 7550 5150 7550
-Wire Wire Line
-	8500 4700 8250 4700
-Wire Wire Line
-	8250 4700 8100 4700
+	8500 4700 8500 4650
+Wire Wire Line
+	3500 7550 5150 7550
+Wire Wire Line
+	8100 4700 8650 4700
 Connection ~ 8500 4700
 Wire Wire Line
 	8650 5450 8650 5350
 Wire Wire Line
-	8100 5350 8100 5200
-Wire Wire Line
-	8100 5200 8100 5100
-Wire Wire Line
-	8100 5100 8100 4900
+	8100 4900 8100 5350
 Connection ~ 8100 5200
 Connection ~ 8500 5200
@@
 	8800 4650 8800 5150
 Wire Wire Line
-	8800 5150 8900 5150
-Wire Wire Line
-	8900 5150 9150 5150
-Wire Wire Line
-	9150 5150 9150 4200
-Wire Wire Line
-	9150 4200 9150 4150
+	8800 5150 9200 5150
 Connection ~ 8900 5150
-Connection ~ 9150 4200
-Wire Wire Line
-	9150 4200 9300 4200
 Connection ~ 8650 5350
 Wire Wire Line
 	8750 6350 8800 6350
 Wire Wire Line
-	10250 6350 10250 5350
-Wire Wire Line
-	10250 5350 10250 4950
+	10250 4950 10250 6350
 Wire Wire Line
 	10250 6350 9300 6350
 Wire Wire Line
-	8100 5350 8650 5350
-Wire Wire Line
-	8650 5350 9250 5350
+	8100 5350 9250 5350
 Wire Wire Line
 	9250 5350 9250 4950
@@
 Connection ~ 10250 5350
 Wire Wire Line
-	3500 7050 3800 7050
-Wire Wire Line
-	3800 7050 3850 7050
+	3500 7050 3850 7050
 Wire Wire Line
 	8100 4700 8100 4600
@@
 Wire Wire Line
 	10250 5350 10350 5350
-Wire Wire Line
-	8100 5100 8250 5100
-Connection ~ 8100 5100
 Connection ~ 8100 4700
 Wire Wire Line
@@
 	9100 6100 9900 6100
 Wire Wire Line
-	9750 2450 9050 2450
-Wire Wire Line
-	9050 2450 8500 2450
+	8500 2450 9750 2450
 Wire Wire Line
 	9050 2500 9050 2450
@@
 Wire Wire Line
 	9050 2900 9050 2950
-Connection ~ 8250 4700
 Wire Wire Line
 	6100 1300 5900 1300
@@
 	4550 3550 6450 3550
 Wire Wire Line
-	5450 1150 5550 1150
-Wire Wire Line
-	5550 1150 5600 1150
+	5450 1150 5600 1150
 Connection ~ 5550 1150
 Wire Wire Line
-	4700 1450 4750 1450
-Wire Wire Line
-	4750 1450 4800 1450
+	4700 1450 4800 1450
 Wire Wire Line
 	5100 1450 5200 1450
@@
 Connection ~ 4500 1050
 Wire Wire Line
-	4700 1250 4750 1250
-Wire Wire Line
-	4750 1250 4900 1250
-Wire Wire Line
-	4900 1250 5050 1250
+	4700 1250 5050 1250
 Wire Wire Line
 	5050 1250 5050 1150
@@
 	13150 2350 13150 2250
 Wire Wire Line
-	14250 1950 14350 1950
-Wire Wire Line
-	14350 1950 14600 1950
-Wire Wire Line
-	14600 1950 14850 1950
-Wire Wire Line
-	14850 1950 15150 1950
-Wire Wire Line
-	14850 1900 14850 1950
-Wire Wire Line
-	14850 1950 14850 2050
+	14250 1950 15150 1950
+Wire Wire Line
+	14850 1900 14850 2050
 Wire Wire Line
 	14850 2400 14850 2350
@@
 Connection ~ 13150 1950
 Wire Wire Line
-	12600 1950 12900 1950
-Wire Wire Line
-	12900 1950 13150 1950
-Wire Wire Line
-	13150 1950 13350 1950
-Wire Wire Line
-	13350 1950 13400 1950
+	12600 1950 13400 1950
 Wire Wire Line
 	12600 2150 12750 2150
@@
 Connection ~ 14600 1950
 Wire Wire Line
-	14450 1900 14450 2050
-Wire Wire Line
-	14450 2050 14450 2200
+	14450 1900 14450 2200
 Wire Wire Line
 	11450 1750 11450 1350
@@
 	13000 1850 12600 1850
 Wire Wire Line
-	13000 1450 13000 1650
-Wire Wire Line
-	13000 1650 13000 1850
+	13000 1450 13000 1850
 Wire Wire Line
 	12800 1000 12900 1000
@@
 	3300 3750 3150 3750
 Wire Wire Line
-	13300 1850 13300 1750
-Wire Wire Line
-	13300 1750 13300 1650
+	13300 1650 13300 1850
 Connection ~ 13300 1750
 Connection ~ 13000 1650
@@
 	14350 2450 14350 1950
 Connection ~ 14350 1950
+Wire Wire Line
+	8650 4700 8650 4750
+Wire Wire Line
+	9150 4150 9200 4150
+Wire Wire Line
+	9200 4150 9200 5150
+$Comp
+L GND #PWR?
+U 1 1 58575B8A
+P 9300 4400
+F 0 "#PWR?" H 9300 4150 50  0001 C CNN
+F 1 "GND" H 9300 4250 50  0000 C CNN
+F 2 "" H 9300 4400 50  0000 C CNN
+F 3 "" H 9300 4400 50  0000 C CNN
+	1    9300 4400
+	0    -1   -1   0
+$EndComp
+Wire Wire Line
+	9300 4400 9200 4400
+Connection ~ 9200 4400
+Wire Wire Line
+	9150 4200 9600 4200
+Wire Wire Line
+	9600 4200 9600 2450
+Connection ~ 9600 2450
 $EndSCHEMATC

Commit message: Initial pcb routing
Parts:
- added C33, C34: C, Capacitors_SMD:C_0805, symbol C
- added P5: BNC, footprints:U.FL-Coax, symbol BNC
- added P6: CONN_01X03, Pin_Headers:Pin_Header_Straight_1x03_Pitch2.54mm, symbol CONN_01X03
- added R28: R, Resistors_SMD:R_0805, symbol R
Connections:
- wire segments 240 -> 244
Changed lines of the file:
@@
 Text GLabel 3300 3000 2    51   Input ~ 0
 MISO
-Text GLabel 3300 2800 2    51   Input ~ 0
+Text GLabel 3300 3650 2    51   Input ~ 0
 DPTT
 Text GLabel 1700 1750 0    51   Input ~ 0
@@
 $EndComp
 $Comp
-L +BATT #PWR033
+L +BATT #PWR032
 U 1 1 582A6C3F
 P 8150 4400
-F 0 "#PWR033" H 8150 4350 20  0001 C CNN
+F 0 "#PWR032" H 8150 4350 20  0001 C CNN
 F 1 "+BATT" H 8150 4500 30  0000 C CNN
 F 2 "" H 8150 4400 60  0000 C CNN
@@
 $EndComp
 $Comp
-L GND-RESCUE-bttnc2 #PWR034
+L GND-RESCUE-bttnc2 #PWR033
 U 1 1 582A7576
 P 10350 5350
-F 0 "#PWR034" H 10350 5350 30  0001 C CNN
+F 0 "#PWR033" H 10350 5350 30  0001 C CNN
 F 1 "GND" H 10350 5280 30  0001 C CNN
 F 2 "" H 10350 5350 60  0000 C CNN
@@
 $EndComp
 $Comp
-L GND-RESCUE-bttnc2 #PWR035
+L GND-RESCUE-bttnc2 #PWR034
 U 1 1 582B609C
 P 9050 2950
-F 0 "#PWR035" H 9050 2950 30  0001 C CNN
+F 0 "#PWR034" H 9050 2950 30  0001 C CNN
 F 1 "GND" H 9050 2880 30  0001 C CNN
 F 2 "" H 9050 2950 60  0000 C CNN
@@
 $EndComp
 $Comp
-L VCC #PWR036
+L VCC #PWR035
 U 1 1 583B6768
 P 5550 850
-F 0 "#PWR036" H 5550 700 50  0001 C CNN
+F 0 "#PWR035" H 5550 700 50  0001 C CNN
 F 1 "VCC" H 5550 1000 50  0000 C CNN
 F 2 "" H 5550 850 50  0000 C CNN
@@
 $EndComp
 $Comp
-L GND #PWR037
+L GND #PWR036
 U 1 1 583ECE2F
 P 4500 1650
-F 0 "#PWR037" H 4500 1400 50  0001 C CNN
+F 0 "#PWR036" H 4500 1400 50  0001 C CNN
 F 1 "GND" H 4500 1500 50  0000 C CNN
 F 2 "" H 4500 1650 50  0000 C CNN
@@
 $EndComp
 $Comp
-L VCC #PWR038
+L VCC #PWR037
 U 1 1 583ECEDB
 P 4500 1000
-F 0 "#PWR038" H 4500 850 50  0001 C CNN
+F 0 "#PWR037" H 4500 850 50  0001 C CNN
 F 1 "VCC" H 4500 1150 50  0000 C CNN
 F 2 "" H 4500 1000 50  0000 C CNN
@@
 $EndComp
 $Comp
-L VCC #PWR039
+L VCC #PWR038
 U 1 1 583EF1E1
 P 5050 850
-F 0 "#PWR039" H 5050 700 50  0001 C CNN
+F 0 "#PWR038" H 5050 700 50  0001 C CNN
 F 1 "VCC" H 5050 1000 50  0000 C CNN
 F 2 "" H 5050 850 50  0000 C CNN
@@
 $EndComp
 $Comp
-L GND #PWR040
+L GND #PWR039
 U 1 1 583EF28F
 P 4900 850
-F 0 "#PWR040" H 4900 600 50  0001 C CNN
+F 0 "#PWR039" H 4900 600 50  0001 C CNN
 F 1 "GND" H 4900 700 50  0000 C CNN
 F 2 "" H 4900 850 50  0000 C CNN
@@
 $EndComp
 $Comp
-L GND #PWR041
+L GND #PWR040
 U 1 1 583F0377
 P 4100 1050
-F 0 "#PWR041" H 4100 800 50  0001 C CNN
+F 0 "#PWR040" H 4100 800 50  0001 C CNN
 F 1 "GND" H 4100 900 50  0000 C CNN
 F 2 "" H 4100 1050 50  0000 C CNN
@@
 $EndComp
 $Comp
-L GND #PWR042
+L GND #PWR041
 U 1 1 5843A819
 P 13400 2600
-F 0 "#PWR042" H 13400 2350 50  0001 C CNN
+F 0 "#PWR041" H 13400 2350 50  0001 C CNN
 F 1 "GND" H 13400 2450 50  0000 C CNN
 F 2 "" H 13400 2600 50  0000 C CNN
@@
 $EndComp
 $Comp
-L GND #PWR043
+L GND #PWR042
 U 1 1 5843CDC2
 P 12900 2350
-F 0 "#PWR043" H 12900 2100 50  0001 C CNN
+F 0 "#PWR042" H 12900 2100 50  0001 C CNN
 F 1 "GND" H 12900 2200 50  0000 C CNN
 F 2 "" H 12900 2350 50  0000 C CNN
@@
 $EndComp
 $Comp
-L GND #PWR044
+L GND #PWR043
 U 1 1 5843D132
 P 13150 2350
-F 0 "#PWR044" H 13150 2100 50  0001 C CNN
+F 0 "#PWR043" H 13150 2100 50  0001 C CNN
 F 1 "GND" H 13150 2200 50  0000 C CNN
 F 2 "" H 13150 2350 50  0000 C CNN
@@
 $EndComp
 $Comp
-L GND #PWR045
+L GND #PWR044
 U 1 1 58440374
 P 14850 2400
-F 0 "#PWR045" H 14850 2150 50  0001 C CNN
+F 0 "#PWR044" H 14850 2150 50  0001 C CNN
 F 1 "GND" H 14850 2250 50  0000 C CNN
 F 2 "" H 14850 2400 50  0000 C CNN
@@
 $EndComp
 $Comp
-L +BATT #PWR046
+L +BATT #PWR045
 U 1 1 58440D22
 P 14850 1900
-F 0 "#PWR046" H 14850 1750 50  0001 C CNN
+F 0 "#PWR045" H 14850 1750 50  0001 C CNN
 F 1 "+BATT" H 14850 2040 50  0000 C CNN
 F 2 "" H 14850 1900 50  0000 C CNN
@@
 $EndComp
 $Comp
-L GND #PWR047
+L GND #PWR046
 U 1 1 58443570
 P 12600 2050
-F 0 "#PWR047" H 12600 1800 50  0001 C CNN
+F 0 "#PWR046" H 12600 1800 50  0001 C CNN
 F 1 "GND" H 12600 1900 50  0000 C CNN
 F 2 "" H 12600 2050 50  0000 C CNN
@@
 GPS_RESET
 $Comp
-L GND #PWR048
+L GND #PWR047
 U 1 1 584518EE
 P 11450 2250
-F 0 "#PWR048" H 11450 2000 50  0001 C CNN
+F 0 "#PWR047" H 11450 2000 50  0001 C CNN
 F 1 "GND" H 11450 2100 50  0000 C CNN
 F 2 "" H 11450 2250 50  0000 C CNN
@@
 $EndComp
 $Comp
-L GND #PWR049
+L GND #PWR048
 U 1 1 58465E84
 P 13300 1750
-F 0 "#PWR049" H 13300 1500 50  0001 C CNN
+F 0 "#PWR048" H 13300 1500 50  0001 C CNN
 F 1 "GND" H 13300 1600 50  0000 C CNN
 F 2 "" H 13300 1750 50  0000 C CNN
@@
 $EndComp
 $Comp
-L +BATT #PWR050
+L +BATT #PWR049
 U 1 1 58466EC9
 P 13600 1450
-F 0 "#PWR050" H 13600 1300 50  0001 C CNN
+F 0 "#PWR049" H 13600 1300 50  0001 C CNN
 F 1 "+BATT" V 13600 1700 50  0000 C CNN
 F 2 "" H 13600 1450 50  0000 C CNN
@@
 $EndComp
 $Comp
-L GND #PWR051
+L GND #PWR050
 U 1 1 58469A68
 P 12300 1000
-F 0 "#PWR051" H 12300 750 50  0001 C CNN
+F 0 "#PWR050" H 12300 750 50  0001 C CNN
 F 1 "GND" H 12300 850 50  0000 C CNN
 F 2 "" H 12300 1000 50  0000 C CNN
@@
 $EndComp
 $Comp
-L GND #PWR052
+L GND #PWR051
 U 1 1 5855596B
 P 8650 5150
-F 0 "#PWR052" H 8650 4900 50  0001 C CNN
+F 0 "#PWR051" H 8650 4900 50  0001 C CNN
 F 1 "GND" H 8650 5000 50  0000 C CNN
 F 2 "" H 8650 5150 50  0000 C CNN
@@
 	3300 2900 3150 2900
 Wire Wire Line
-	3150 2800 3300 2800
-Wire Wire Line
 	3150 3450 3300 3450
 Wire Wire Line
@@
 	9200 4150 9200 5150
 $Comp
-L GND #PWR?
+L GND #PWR052
 U 1 1 58575B8A
 P 9300 4400
-F 0 "#PWR?" H 9300 4150 50  0001 C CNN
+F 0 "#PWR052" H 9300 4150 50  0001 C CNN
 F 1 "GND" H 9300 4250 50  0000 C CNN
 F 2 "" H 9300 4400 50  0000 C CNN
@@
 	9600 4200 9600 2450
 Connection ~ 9600 2450
+$Comp
+L R R28
+U 1 1 58990409
+P 10950 2150
+F 0 "R28" V 11030 2150 50  0000 C CNN
+F 1 "R" V 10950 2150 50  0000 C CNN
+F 2 "Resistors_SMD:R_0805" V 10880 2150 50  0001 C CNN
+F 3 "" H 10950 2150 50  0000 C CNN
+	1    10950 2150
+	0    1    1    0
+$EndComp
+$Comp
+L C C34
+U 1 1 58990514
+P 11150 2300
+F 0 "C34" H 10950 2200 50  0000 L CNN
+F 1 "C" H 11175 2200 50  0000 L CNN
+F 2 "Capacitors_SMD:C_0805" H 11188 2150 50  0001 C CNN
+F 3 "" H 11150 2300 50  0000 C CNN
+	1    11150 2300
+	1    0    0    -1
+$EndComp
+$Comp
+L C C33
+U 1 1 589908B9
+P 10750 2300
+F 0 "C33" H 10600 2200 50  0000 L CNN
+F 1 "C" H 10775 2200 50  0000 L CNN
+F 2 "Capacitors_SMD:C_0805" H 10788 2150 50  0001 C CNN
+F 3 "" H 10750 2300 50  0000 C CNN
+	1    10750 2300
+	1    0    0    -1
+$EndComp
+$Comp
+L BNC P5
+U 1 1 589909AC
+P 10500 2150
+F 0 "P5" H 10510 2270 50  0000 C CNN
+F 1 "BNC" V 10610 2090 50  0000 C CNN
+F 2 "footprints:U.FL-Coax" H 10500 2150 50  0001 C CNN
+F 3 "" H 10500 2150 50  0000 C CNN
+	1    10500 2150
+	-1   0    0    -1
+$EndComp
+Wire Wire Line
+	10650 2150 10800 2150
+Wire Wire Line
+	11100 2150 11450 2150
+Connection ~ 10750 2150
+Connection ~ 11150 2150
+$Comp
+L GND #PWR053
+U 1 1 58991ACA
+P 10500 2350
+F 0 "#PWR053" H 10500 2100 50  0001 C CNN
+F 1 "GND" H 10500 2200 50  0000 C CNN
+F 2 "" H 10500 2350 50  0000 C CNN
+F 3 "" H 10500 2350 50  0000 C CNN
+	1    10500 2350
+	1    0    0    -1
+$EndComp
+$Comp
+L GND #PWR054
+U 1 1 58991CF0
+P 10750 2450
+F 0 "#PWR054" H 10750 2200 50  0001 C CNN
+F 1 "GND" H 10750 2300 50  0000 C CNN
+F 2 "" H 10750 2450 50  0000 C CNN
+F 3 "" H 10750 2450 50  0000 C CNN
+	1    10750 2450
+	1    0    0    -1
+$EndComp
+$Comp
+L GND #PWR055
+U 1 1 58991F1A
+P 11150 2450
+F 0 "#PWR055" H 11150 2200 50  0001 C CNN
+F 1 "GND" H 11150 2300 50  0000 C CNN
+F 2 "" H 11150 2450 50  0000 C CNN
+F 3 "" H 11150 2450 50  0000 C CNN
+	1    11150 2450
+	1    0    0    -1
+$EndComp
+$Comp
+L CONN_01X03 P6
+U 1 1 589928AC
+P 6700 7250
+F 0 "P6" H 6700 7450 50  0000 C CNN
+F 1 "CONN_01X03" V 6800 7250 50  0000 C CNN
+F 2 "Pin_Headers:Pin_Header_Straight_1x03_Pitch2.54mm" H 6700 7250 50  0001 C CNN
+F 3 "" H 6700 7250 50  0000 C CNN
+	1    6700 7250
+	1    0    0    1
+$EndComp
+$Comp
+L GND #PWR056
+U 1 1 58993DB6
+P 6450 7400
+F 0 "#PWR056" H 6450 7150 50  0001 C CNN
+F 1 "GND" H 6450 7250 50  0000 C CNN
+F 2 "" H 6450 7400 50  0000 C CNN
+F 3 "" H 6450 7400 50  0000 C CNN
+	1    6450 7400
+	1    0    0    -1
+$EndComp
+Wire Wire Line
+	6450 7400 6450 7350
+Wire Wire Line
+	6450 7350 6500 7350
+Text GLabel 6500 7150 0    48   Input ~ 0
+RXD
+Text GLabel 6500 7250 0    48   Input ~ 0
+TXD
+Wire Wire Line
+	3150 3650 3300 3650
 $EndSCHEMATC

Commit message: Update and rearrange labels
Parts:
- P3: value BNC -> SMA
- P5: value BNC -> U.FL
- P6: value CONN_01X03 -> Serial
Other:
- moved on the sheet: C1, C10, C11, C12, C13, C14, C15, C16, C17, C18, C19, C2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
